Commit message: added d01 model

File: src/diff_wheeled_robot_gazebo/urdf/VLP-16.urdf.xacro (robot description, xacro)
@@ -18,10 +18,10 @@
       <visual>
         <geometry>
-          <mesh filename="package://velodyne_description/meshes/VLP16_base_1.dae" />
+          <mesh filename="package://diff_wheeled_robot_gazebo/meshes/VLP16_base_1.dae" />
         </geometry>
       </visual>
       <visual>
         <geometry>
-          <mesh filename="package://velodyne_description/meshes/VLP16_base_2.dae" />
+          <mesh filename="package://diff_wheeled_robot_gazebo/meshes/VLP16_base_2.dae" />
         </geometry>
       </visual>
@@ -47,5 +47,5 @@
         <origin xyz="0 0 -0.0377" />
         <geometry>
-          <mesh filename="package://velodyne_description/meshes/VLP16_scan.dae" />
+          <mesh filename="package://diff_wheeled_robot_gazebo/meshes/VLP16_scan.dae" />
         </geometry>
       </visual>

File: src/diff_wheeled_robot_gazebo/urdf/diff_wheeled_robot.xacro (robot description, xacro)
@@ -184,5 +184,5 @@
       <broadcastTF>1</broadcastTF>
       <wheelTorque>30</wheelTorque>
-      <wheelAcceleration>1.8</wheelAcceleration>
+      <wheelAcceleration>2.5</wheelAcceleration>
       <commandTopic>cmd_vel</commandTopic>
       <odometryFrame>odom</odometryFrame>

File: src/diff_wheeled_robot_gazebo/urdf/diff_wheeled_robot_with_vlp_16.xacro (robot description, xacro)
@@ -5,8 +5,10 @@
   <xacro:arg name="organize_cloud" default="false"/>
   <xacro:property name="organize_cloud" value="$(arg organize_cloud)" />
+  <xacro:property name="base_radius_velodyne" value="0.0516"/>
   <xacro:include filename="$(find diff_wheeled_robot_gazebo)/urdf/diff_wheeled_robot.xacro" />
   <xacro:include filename="$(find velodyne_description)/urdf/VLP-16.urdf.xacro"/>
   <xacro:VLP-16 parent="base_link" name="velodyne" topic="/velodyne_points" organize_cloud="${organize_cloud}" hz="10" samples="440" gpu="${gpu}">
-    <origin xyz="${base_radius - hokuyo_size/2} 0 ${base_height+hokuyo_size/8}" rpy="0 0 0" />
+    <!--origin xyz="${base_radius - base_radius_velodyne} 0 ${base_height/2}" rpy="0 0 0" /-->
+   <origin xyz="0 0 ${base_height/2}" rpy="0 0 0" />
   </xacro:VLP-16>
 </robot>

Commit message: fixed navigation error due to oscillation and modified some parameter of car model

File: src/diff_wheeled_robot_gazebo/urdf/VLP-16.urdf.xacro (robot description, xacro)
@@ -2,5 +2,5 @@
 <robot xmlns:xacro="http://www.ros.org/wiki/xacro" name="VLP-16">
   <xacro:property name="M_PI" value="3.1415926535897931" />
-  <xacro:macro name="VLP-16" params="*origin parent:=base_link name:=velodyne topic:=/velodyne_points organize_cloud:=false hz:=10 lasers:=16 samples:=1875 collision_range:=0.3 min_range:=0.9 max_range:=130.0 noise:=0.008 min_angle:=-${M_PI} max_angle:=${M_PI} gpu:=false">
+  <xacro:macro name="VLP-16" params="*origin parent:=base_link name:=velodyne topic:=/velodyne_points organize_cloud:=false hz:=10 lasers:=16 samples:=1875 collision_range:=0.03 min_range:=0.05 max_range:=130.0 noise:=0.008 min_angle:=-${M_PI} max_angle:=${M_PI} gpu:=false">
     <joint name="${name}_base_mount_joint" type="fixed">
       <xacro:insert_block name="origin" />

File: src/diff_wheeled_robot_gazebo/urdf/d01/d01.urdf.xacro (robot description, xacro)
@@ -118,8 +118,10 @@
         <xacro:action_wheel parent="base_link" name="rightfront" radius="0.7" length="0.3" flipY="-1" translateX="0.8" translateY="0.9">
         </xacro:action_wheel>
+        <!-->
         <xacro:action_wheel parent="base_link" name="leftback" radius="0.7" length="0.3" flipY="-1" translateX="-0.8" translateY="-0.9">
         </xacro:action_wheel>
         <xacro:action_wheel parent="base_link" name="rightback" radius="0.7" length="0.3" flipY="-1" translateX="-0.8" translateY="0.9">
         </xacro:action_wheel>
+<-->
         <gazebo>
             <plugin name="differential_drive_controller" filename="libgazebo_ros_diff_drive.so">
@@ -144,7 +146,7 @@
             </plugin>
         </gazebo>
-<xacro:property name="laser_plattform_width" value="0.12"/>
-<xacro:property name="laser_plattform_length" value="0.12"/>
-<xacro:property name="laser_plattform_height" value="0.6"/>
+        <xacro:property name="laser_plattform_width" value="0.12"/>
+        <xacro:property name="laser_plattform_length" value="0.12"/>
+        <xacro:property name="laser_plattform_height" value="0.6"/>
         <link name="laser_plattform_link">
             <visual>
@@ -179,3 +181,24 @@
             <origin xyz="0 0 ${laser_plattform_height/2}" rpy="0 0 0" />
         </xacro:VLP-16>
+        <xacro:include filename="$(find diff_wheeled_robot_gazebo)/urdf/d01/d01_driven_wheel.urdf.xacro"/>
+        <!--
+        <xacro:castor_mount parent="base_link" name="left"  base_x_origin_to_castor_mount_origin="1.01" base_y_origin_to_castor_mount_origin="0.85" base_z_origin_to_castor_mount_origin="-0.65" translateX="-1" translateY="1">
+        </xacro:castor_mount>
+        <xacro:castor_mount parent="base_link" name="right"  base_x_origin_to_castor_mount_origin="1.01" base_y_origin_to_castor_mount_origin="0.85" base_z_origin_to_castor_mount_origin="-0.65" translateX="-1" translateY="-1">
+        </xacro:castor_mount>
+        <xacro:castor_dummy  parent="left_castor_mount_link" name="left">
+        </xacro:castor_dummy>
+        <xacro:castor_dummy  parent="right_castor_mount_link" name="right">
+        </xacro:castor_dummy>
+        <xacro:driven_wheel parent="left_castor_mount_link" name="left" radius="0.25" length="0.2">
+        </xacro:driven_wheel>
+          <xacro:driven_wheel parent="right_castor_mount_link" name="right" radius="0.25" length="0.2">
+        </xacro:driven_wheel>
+    -->
+    <xacro:driven_wheel_sphere parent="base_link" name="left" radius="0.6" base_x_origin_to_wheel_origin="1.01" base_y_origin_to_wheel_origin="0" base_z_origin_to_wheel_origin="-0.6" translateX="-1" translateY="-1">
+    </xacro:driven_wheel_sphere>
+    <!--
+    <xacro:driven_wheel_sphere parent="base_link" name="right" radius="0.6" base_x_origin_to_wheel_origin="1.01" base_y_origin_to_wheel_origin="0.85" base_z_origin_to_wheel_origin="-0.6" translateX="-1" translateY="1">
+    </xacro:driven_wheel_sphere>
+    -->
     </robot>

File: src/diff_wheeled_robot_gazebo/urdf/d01/d01_driven_wheel.urdf.xacro (robot description, xacro)
@@ -1,5 +1,135 @@
 <?xml version="1.0"?>
 <robot xmlns:xacro="http://www.ros.org/wiki/xacro" name="driven_wheel">
-    <xacro:macro name="driven_wheel" params="">
+    <xacro:property name="castor_mount_link_length" value="0.1145"/>
+    <xacro:property name="castor_mount_link_width" value=" 0.10"/>
+    <xacro:property name="castor_mount_link_height" value=" 0.0057"/>
+    <xacro:property name="castor_dummy_link_length" value="0.02"/>
+    <xacro:property name="castor_dummy_link_width" value="0.02"/>
+    <xacro:property name="castor_dummy_link_height" value="0.02"/>
+    <xacro:macro name="castor_mount" params="parent name base_x_origin_to_castor_mount_origin base_y_origin_to_castor_mount_origin base_z_origin_to_castor_mount_origin translateX translateY">
+        <link name="${name}_castor_mount_link">
+            <visual>
+                <origin xyz="0.0 0.0 0" rpy="0.0 0 0.0"/>
+                <geometry>
+                    <box size="${castor_mount_link_length} ${castor_mount_link_width} ${castor_mount_link_height}"/>
+                </geometry>
+            </visual>
+            <collision>
+                <origin xyz="0.0 0.0 0" rpy="0.0 0 0.0"/>
+                <geometry>
+                    <box size="${castor_mount_link_length} ${castor_mount_link_width} ${castor_mount_link_height}"/>
+                </geometry>
+            </collision>
+            <inertial>
+                <origin xyz="0.0 0.0 0" rpy="0.0 0 0.0"/>
+                <mass value="1"/>
+                <inertia ixx="1" ixy="0.0" ixz="0.0" iyy="1" iyz="0.0" izz="1"/>
+            </inertial>
+        </link>
+        <joint name="${name}_castor_mount_joint" type="fixed">
+            <parent link="${parent}"/>
+            <child link="${name}_castor_mount_link"/>
+            <origin xyz="${base_x_origin_to_castor_mount_origin*translateX} ${base_y_origin_to_castor_mount_origin*translateY} ${base_z_origin_to_castor_mount_origin}" rpy="0.0 0.0 0.0"/>
+        </joint>
+        <gazebo reference="${name}_castor_mount_link">
+            <material>Gazebo/White</material>
+            <turnGravityOff>false</turnGravityOff>
+        </gazebo>
+    </xacro:macro>
+    <xacro:macro name="castor_dummy" params="parent name">
+        <link name="${name}_castor_dummy_link">
+            <visual>
+                <origin xyz="0 0 0.0" rpy="0.0 0.0 0.0"/>
+                <geometry>
+                    <box size="${castor_dummy_link_width} ${castor_dummy_link_length} ${castor_dummy_link_height}"/>
+                </geometry>
+            </visual>
+            <collision>
+                <origin xyz="0 0 0.0" rpy="0.0 0.0 0.0"/>
+                <geometry>
+                    <box size="${castor_dummy_link_width} ${castor_dummy_link_length} ${castor_dummy_link_height}"/>
+                </geometry>
+            </collision>
+            <inertial>
+                <origin xyz="0 0 0.0" rpy="0.0 0.0 0.0"/>
+                <mass value="1"/>
+                <inertia ixx="1" ixy="0.0" ixz="0.0" iyy="1" iyz="0.0" izz="1"/>
+            </inertial>
+        </link>
+        <joint name="${name}_castor_dummy_joint" type="continuous">
+            <parent link="${parent}"/>
+            <child link="${name}_castor_dummy_link"/>
+            <axis xyz="0 0 1"/>
+            <origin xyz="0 0 -0.05" rpy="0 0 0"/>
+            <limit effort="100" velocity="100"/>
+            <joint_properties damping="0.0" friction="1.5"/>
+        </joint>
+        <gazebo reference="${name}_castor_dummy_link">
+            <material>Gazebo/White</material>
+            <turnGravityOff>false</turnGravityOff>
+        </gazebo>
+    </xacro:macro>
+    <xacro:macro name="driven_wheel" params="parent name radius length">
+        <link name="${name}_driven_wheel_link">
+            <visual>
+                <origin xyz="0.0 0.0 ${-radius}" rpy="${M_PI/2} 0 0.0"/>
+                <geometry>
+                    <cylinder radius="${radius}" length="${length}"/>
+                </geometry>
+            </visual>
+            <collision>
+                <origin xyz="0.0 0.0 ${-radius}" rpy="${M_PI/2} 0 0.0"/>
+                <geometry>
+                    <cylinder radius="${radius}" length="${length}"/>
+                </geometry>
+            </collision>
+            <inertial>
+                <origin xyz="0.0 0.0 ${-radius}" rpy="${M_PI/2} 0 0.0"/>
+                <mass value="1"/>
+                <inertia ixx="1" ixy="0.0" ixz="0.0" iyy="1" iyz="0.0" izz="1"/>
+            </inertial>
+        </link>
+        <joint name="${name}_driven_wheel_joint" type="continuous">
+            <parent link="${parent}"/>
+            <child link="${name}_driven_wheel_link"/>
+            <axis xyz="0 1 0"/>
+            <origin xyz="0 0 -0.1" rpy="0 0 0"/>
+            <limit effort="100" velocity="100"/>
+            <joint_properties damping="0.0" friction="1.5"/>
+        </joint>
+        <gazebo reference="${name}_castor_dummy_link">
+            <material>Gazebo/Black</material>
+            <turnGravityOff>false</turnGravityOff>
+        </gazebo>
+    </xacro:macro>
+    <xacro:macro name="driven_wheel_sphere" params="name parent radius base_x_origin_to_wheel_origin base_y_origin_to_wheel_origin base_z_origin_to_wheel_origin translateX translateY">
+        <link name="${name}_driven_wheel_sphere_link">
+            <visual>
+                <origin xyz="0.0 0.0 0.0" rpy="0.0 0.0 0.0"/>
+                <geometry>
+                    <sphere radius="${radius}"/>
+                </geometry>
+            </visual>
+            <collision>
+                <origin xyz="0.0 0.0 0.0" rpy="0.0 0.0 0.0"/>
+                <geometry>
+                    <sphere radius="${radius}"/>
+                </geometry>
+            </collision>
+            <inertial>
+                <origin xyz="0.0 0.0 0.0" rpy="0.0 0.0 0.0"/>
+                <mass value="1"/>
+                <inertia ixx="1" ixy="0.0" ixz="0" iyy="1" iyz="0.0" izz="1"/>
+            </inertial>
+        </link>
+        <joint name="${name}_driven_wheel_sphere_joint" type="fixed">
+            <parent link="${parent}"/>
+            <child link="${name}_driven_wheel_sphere_link"/>
+            <origin xyz="${base_x_origin_to_wheel_origin*translateX} ${base_y_origin_to_wheel_origin*translateY} ${base_z_origin_to_wheel_origin}" rpy="0.0 0.0 0.0"/>
+        </joint>
+        <gazebo reference="${name}_driven_wheel_sphere_link">
+            <material>Gazebo/Black</material>
+            <turnGravityOff>false</turnGravityOff>
+        </gazebo>
     </xacro:macro>
 </robot>

File: src/diff_wheeled_robot_gazebo/urdf/diff_wheeled_robot.xacro (robot description, xacro)
@@ -28,10 +28,10 @@
   <!-- caster wheel mass -->
   <xacro:property name="caster_f_height" value="0.04" />
-  <xacro:property name="caster_f_radius" value="0.025" />
+  <xacro:property name="caster_f_radius" value="0.028" />
   <xacro:property name="caster_f_mass" value="0.5" /> <!-- in kg-->
   <!-- caster wheel radius and height -->
   <!-- caster wheel mass -->
   <xacro:property name="caster_b_height" value="0.04" />
-  <xacro:property name="caster_b_radius" value="0.025" />
+  <xacro:property name="caster_b_radius" value="0.0275" />
   <xacro:property name="caster_b_mass" value="0.5" /> <!-- in kg-->
   <!-- Wheels -->
@@ -183,7 +183,7 @@
       <wheelDiameter>${2*wheel_radius}</wheelDiameter>
       <broadcastTF>1</broadcastTF>
-      <wheelTorque>30</wheelTorque>
+      <wheelTorque>100</wheelTorque>
       <wheelAcceleration>2.5</wheelAcceleration>
-      <commandTopic>cmd_vel</commandTopic>
+      <commandTopic>/cmd_vel</commandTopic>
       <odometryFrame>odom</odometryFrame>
       <odometryTopic>odom</odometryTopic>

File: src/diff_wheeled_robot_gazebo/urdf/diff_wheeled_robot_with_vlp_16.xacro (robot description, xacro)
@@ -10,5 +10,5 @@
   <xacro:VLP-16 parent="base_link" name="velodyne" topic="/velodyne_points" organize_cloud="${organize_cloud}" hz="10" samples="440" gpu="${gpu}">
     <!--origin xyz="${base_radius - base_radius_velodyne} 0 ${base_height/2}" rpy="0 0 0" /-->
-   <origin xyz="0 0 ${base_height/2}" rpy="0 0 0" />
+   <origin xyz="${base_radius - base_radius_velodyne} 0 ${base_height/2}" rpy="0 0 0" />
   </xacro:VLP-16>
 </robot>

File: src/diff_wheeled_robot_gazebo/urdf/wheel.urdf.xacro (robot description, xacro)
@@ -35,6 +35,6 @@
     </link>
     <gazebo reference="${fb}_${lr}_wheel">
-      <mu1 value="1.0"/>
-      <mu2 value="1.0"/>
+      <mu1 value="10000000"/>
+      <mu2 value="10000000"/>
       <kp  value="10000000.0" />
       <kd  value="1.0" />
@@ -48,5 +48,5 @@
       <origin xyz="${translateX * base_x_origin_to_wheel_origin} ${translateY * base_y_origin_to_wheel_origin} ${base_z_origin_to_wheel_origin}" rpy="0 0 0" />
       <axis xyz="0 1 0" rpy="0  0" />
-      <limit effort="100" velocity="100"/>
+      <limit effort="1000" velocity="100"/>
       <joint_properties damping="0.0" friction="0.0"/>
     </joint>
